Commit message: Pushed a lot the pid values; it seems this is the maximum

File: data/robots/soft_hand.urdf (robot description, URDF)
Before this commit: robot soft_hand, 39 links, 38 joints
Links:
- link soft_hand_index_distal_link: mass 0.1 -> 0.1*0.01
- link soft_hand_index_fake_link1: mass 0.1 -> 0.1*0.01
- link soft_hand_index_fake_link2: mass 0.1 -> 0.1*0.01
- link soft_hand_index_fake_link3: mass 0.1 -> 0.1*0.01
- link soft_hand_index_knuckle_link: mass 0.09 -> 0.09*0.01
- link soft_hand_index_middle_link: mass 0.05 -> 0.05*0.01
- link soft_hand_index_proximal_link: mass 0.05 -> 0.05*0.01
- link soft_hand_invisible_wire_link: mass 0.1 -> 0.1*0.01
- link soft_hand_little_distal_link: mass 0.1 -> 0.1*0.01
- link soft_hand_little_fake_link1: mass 0.1 -> 0.1*0.01
- link soft_hand_little_fake_link2: mass 0.1 -> 0.1*0.01
- link soft_hand_little_fake_link3: mass 0.1 -> 0.1*0.01
- link soft_hand_little_knuckle_link: mass 0.09 -> 0.09*0.01
- link soft_hand_little_middle_link: mass 0.05 -> 0.05*0.01
- link soft_hand_little_proximal_link: mass 0.05 -> 0.05*0.01
- link soft_hand_middle_distal_link: mass 0.1 -> 0.1*0.01
- link soft_hand_middle_fake_link1: mass 0.1 -> 0.1*0.01
- link soft_hand_middle_fake_link2: mass 0.1 -> 0.1*0.01
- link soft_hand_middle_fake_link3: mass 0.1 -> 0.1*0.01
- link soft_hand_middle_knuckle_link: mass 0.09 -> 0.09*0.01
- link soft_hand_middle_middle_link: mass 0.05 -> 0.05*0.01
- link soft_hand_middle_proximal_link: mass 0.05 -> 0.05*0.01
- link soft_hand_palm_link: mass 2.28 -> 2.28*0.01
- link soft_hand_ring_distal_link: mass 0.1 -> 0.1*0.01
- link soft_hand_ring_fake_link1: mass 0.1 -> 0.1*0.01
- link soft_hand_ring_fake_link2: mass 0.1 -> 0.1*0.01
- link soft_hand_ring_fake_link3: mass 0.1 -> 0.1*0.01
- link soft_hand_ring_knuckle_link: mass 0.09 -> 0.09*0.01
- link soft_hand_ring_middle_link: mass 0.05 -> 0.05*0.01
- link soft_hand_ring_proximal_link: mass 0.05 -> 0.05*0.01
- link soft_hand_thumb_distal_link: mass 0.1 -> 0.1*0.01
- link soft_hand_thumb_fake_link1: mass 0.1 -> 0.1*0.01
- link soft_hand_thumb_fake_link3: mass 0.1 -> 0.1*0.01
- link soft_hand_thumb_knuckle_link: mass 0.09 -> 0.09*0.01
- link soft_hand_thumb_proximal_link: mass 0.05 -> 0.05*0.01

Commit message: Unfortunately, with these unrealistic values, simulation seems a lot better...

File: data/robots/soft_hand.urdf (robot description, URDF)
Before this commit: robot soft_hand, 39 links, 38 joints
Links:
- link soft_hand_index_distal_link: mass 0.1*0.01 -> 0.1
- link soft_hand_index_fake_link1: mass 0.1*0.01 -> 0.1
- link soft_hand_index_fake_link2: mass 0.1*0.01 -> 0.1
- link soft_hand_index_fake_link3: mass 0.1*0.01 -> 0.1
- link soft_hand_index_knuckle_link: mass 0.09*0.01 -> 0.09
- link soft_hand_index_middle_link: mass 0.05*0.01 -> 0.05
- link soft_hand_index_proximal_link: mass 0.05*0.01 -> 0.05
- link soft_hand_invisible_wire_link: mass 0.1*0.01 -> 0.1
- link soft_hand_little_distal_link: mass 0.1*0.01 -> 0.1
- link soft_hand_little_fake_link1: mass 0.1*0.01 -> 0.1
- link soft_hand_little_fake_link2: mass 0.1*0.01 -> 0.1
- link soft_hand_little_fake_link3: mass 0.1*0.01 -> 0.1
- link soft_hand_little_knuckle_link: mass 0.09*0.01 -> 0.09
- link soft_hand_little_middle_link: mass 0.05*0.01 -> 0.05
- link soft_hand_little_proximal_link: mass 0.05*0.01 -> 0.05
- link soft_hand_middle_distal_link: mass 0.1*0.01 -> 0.1
- link soft_hand_middle_fake_link1: mass 0.1*0.01 -> 0.1
- link soft_hand_middle_fake_link2: mass 0.1*0.01 -> 0.1
- link soft_hand_middle_fake_link3: mass 0.1*0.01 -> 0.1
- link soft_hand_middle_knuckle_link: mass 0.09*0.01 -> 0.09
- link soft_hand_middle_middle_link: mass 0.05*0.01 -> 0.05
- link soft_hand_middle_proximal_link: mass 0.05*0.01 -> 0.05
- link soft_hand_palm_link: mass 2.28*0.01 -> 2.28
- link soft_hand_ring_distal_link: mass 0.1*0.01 -> 0.1
- link soft_hand_ring_fake_link1: mass 0.1*0.01 -> 0.1
- link soft_hand_ring_fake_link2: mass 0.1*0.01 -> 0.1
- link soft_hand_ring_fake_link3: mass 0.1*0.01 -> 0.1
- link soft_hand_ring_knuckle_link: mass 0.09*0.01 -> 0.09
- link soft_hand_ring_middle_link: mass 0.05*0.01 -> 0.05
- link soft_hand_ring_proximal_link: mass 0.05*0.01 -> 0.05
- link soft_hand_thumb_distal_link: mass 0.1*0.01 -> 0.1
- link soft_hand_thumb_fake_link1: mass 0.1*0.01 -> 0.1
- link soft_hand_thumb_fake_link3: mass 0.1*0.01 -> 0.1
- link soft_hand_thumb_knuckle_link: mass 0.09*0.01 -> 0.09
- link soft_hand_thumb_proximal_link: mass 0.05*0.01 -> 0.05

Commit message: Rotated kuka coupler frame in order to avoid rpy singularities

File: data/robots/soft_hand.urdf (robot description, URDF)
Before this commit: robot soft_hand, 39 links, 38 joints
Joints:
- joint box_soft_hand_kuka_coupler_base_joint: origin xyz=0 0 0.023 rpy=0 0 0 -> xyz=0 0 0.023 rpy=0 0 0.7854
